File: 2017/Motherboard/Motherboard.sch (KiCad schematic (older format))
At the start: 23 parts, among them U1 MSP432, Y1 32.768khz

Commit message: Add Card LEDs to the board
Parts:
- removed U?: AZ117CH-5.0, symbol AZ117CH-5.0
- added D? (x3): LED, symbol LED
- added R? (x3): R, symbol R
- added U?: LM340MP-5.0, SOT-223-4, symbol LM340MP-5.0
Connections:
- net +12V: now also P?.11 (P11), P?.11 (P11), P?.11 (P11), P?.13 (P13), P?.13 (P13), P?.13 (P13), P?.15 (P15), P?.15 (P15), P?.15 (P15), U?.1 (INPUT)
- net +3V3: no longer P?.11 (P11), P?.11 (P11), P?.11 (P11), P?.13 (P13), P?.13 (P13), P?.13 (P13), P?.15 (P15), P?.15 (P15), P?.15 (P15)
- net +5V: now also U?.3 (OUTPUT)
- net GND: now also U?.2 (GND)
- net RX1: now also P?.27 (P27), P?.27 (P27), P?.27 (P27); no longer P?.29 (P29), P?.29 (P29), P?.29 (P29)
- net RX2: now also P?.31 (P31), P?.31 (P31), P?.31 (P31); no longer P?.33 (P33), P?.33 (P33), P?.33 (P33)
- net SCL1: now also P?.21 (P21), P?.21 (P21), P?.21 (P21); no longer P?.23 (P23), P?.23 (P23), P?.23 (P23)
- net SCL2: now also P?.25 (P25), P?.25 (P25), P?.25 (P25); no longer P?.27 (P27), P?.27 (P27), P?.27 (P27)
- net SDA1: now also P?.19 (P19), P?.19 (P19), P?.19 (P19); no longer P?.21 (P21), P?.21 (P21), P?.21 (P21)
- net SDA2: now also P?.23 (P23), P?.23 (P23), P?.23 (P23); no longer P?.25 (P25), P?.25 (P25), P?.25 (P25)
- net TX1: now also P?.29 (P29), P?.29 (P29), P?.29 (P29); no longer P?.31 (P31), P?.31 (P31), P?.31 (P31)
- net TX2: now also P?.33 (P33), P?.33 (P33), P?.33 (P33); no longer P?.35 (P35), P?.35 (P35), P?.35 (P35)
- net at P?.36 (P36): now also R?.1 (x3)
- new net: D?.1 (K), P?.35 (P35) (x3)
- new net: D?.2 (A), R?.2 (x3)
- no-connect marks 0 -> 30
Other:
- note added: "PCIe Cards"
- moved on the sheet: P?

Commit message: Motherboard - Correct PINOUT to match TI pinmux, add HF X, create PCIe_36 footprint, add temperature sensor, create and assign netlist, BOM
Parts:
- removed P?: SWD Programming Header, symbol CONN_01X05
- added C10, C9: 20p, Capacitors_SMD:C_0603, symbol C
- added D6, D7, D8, D9: LED, LEDs:LED_0603, symbol LED
- added P2: PROGRAM+DEBUG, Pin_Headers:Pin_Header_Straight_1x10, symbol CONN_01X10
- added R10, R7, R8, R9: 220, Resistors_SMD:R_1206, symbol R
- added R11, R12, R13, R14, R15, R16: 2.2k, Resistors_SMD:R_0805, symbol R
- added U4: MCP9808, Housings_SSOP:MSOP-8_3x3mm_Pitch0.65mm, symbol MCP9808
- added Y2: 48MHz, symbol Crystal
- C1, C2: footprint (none) -> Capacitors_SMD:C_0603
- C3, C4: value 12.5p -> 22p; footprint (none) -> Capacitors_SMD:C_0603; Digikey (none) -> http://www.digikey.com/product-detail/en/avx-corporation/06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
- C5, C6, C7, C8: renamed from C?; footprint (none) -> Capacitors_SMD:C_0805
- D1: renamed from D?; value LED -> RFD900 PWR LED; footprint (none) -> LEDs:LED_0603
- D2, D3, D4, D5: renamed from D?; footprint (none) -> LEDs:LED_0603
- P1: renamed from P?; value EdgeCard -> DB9; footprint (none) -> Connectors:DB9FD
- P3, P4, P5: renamed from P?; footprint (none) -> Connectors:PCIe_36
- R1, R2, R3: renamed from R?; footprint (none) -> Resistors_SMD:R_0805
- R4, R5, R6: renamed from R?; value R -> 220; footprint (none) -> Resistors_SMD:R_1206
- SW1: renamed from SW?; footprint (none) -> Buttons_Switches_SMD:SW_SPST_EVQP0
- U1: footprint (none) -> Housings_QFP:LQFP-100_14x14mm_Pitch0.5mm
- U2: renamed from U?; footprint SOT-223-4 -> TO_SOT_Packages_SMD:SOT-223
- U3: renamed from U?; value AZ117C-3.3 -> LD1086DT33TR; footprint (none) -> TO_SOT_Packages_SMD:TO-252-2Lead; Digikey http://www.digikey.com/product-detail/en/diodes-incorporate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 -> http://www.digikey.com/product-detail/en/stmicroelectronics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
Connections:
- net +12V: no longer P3.11 (P11), P3.13 (P13), P3.15 (P15), P3.7 (P7), P3.9 (P9), P4.11 (P11), P4.13 (P13), P4.15 (P15), P4.7 (P7), P4.9 (P9), P5.11 (P11), P5.13 (P13), P5.15 (P15), P5.7 (P7), P5.9 (P9)
- net +3V3: now also P3.7 (P7), P3.9 (P9), P4.7 (P7), P4.9 (P9), P5.7 (P7), P5.9 (P9), D6.2 (A), D7.2 (A), D8.2 (A), D9.2 (A), P2.3 (P3), R11.1, R12.1, R13.1, R14.1, R15.1, R16.1, U4.8 (VDD)
- net +5V: now also P3.11 (P11), P3.13 (P13), P4.11 (P11), P4.13 (P13), P5.11 (P11), P5.13 (P13), P2.2 (P2)
- net GND: now also C10.2, C9.2, P2.1 (P1), U4.4 (GND), U4.5 (A2), U4.6 (A1), U4.7 (A0); no longer P3.16 (P16), P4.16 (P16), P5.16 (P16)
- net RSTn: now also P2.6 (P6)
- net RX1: now also P1.2 (P2), U1.23 (P2.7); no longer P3.27 (P27), P4.27 (P27), P5.27 (P27)
- net SCL1: now also P3.29 (P29), P4.29 (P29), P5.29 (P29), U1.79 (P6.5), R16.2; no longer P3.21 (P21), P4.21 (P21), P5.21 (P21)
- net SCL2: now also U1.17 (P2.1), R11.2, U4.2 (SCL); no longer P3.25 (P25), P4.25 (P25), P5.25 (P25)
- net SDA1: now also P3.27 (P27), P4.27 (P27), P5.27 (P27), U1.78 (P6.4), R15.2; no longer P3.19 (P19), P4.19 (P19), P5.19 (P19)
- net SDA2: now also U1.21 (P2.5), R12.2, U4.1 (SDA); no longer P3.23 (P23), P4.23 (P23), P5.23 (P23)
- net SWCLK: now also P2.8 (P8)
- net SWDIO: now also P2.7 (P7)
- net TX1: now also P1.3 (P3), U1.22 (P2.6); no longer P3.29 (P29), P4.29 (P29), P5.29 (P29)
- net UCA0RXD: now also P2.4 (P4); no longer P1.2 (P2)
- net UCA0TXD: now also P2.5 (P5); no longer P1.3 (P3)
- net TestLED1: now reaches U1.26 (P7.4)
- net TestLED1: now also R7.2
- net TestLED2: now reaches U1.27 (P7.5)
- net TestLED2: now also R8.2
- net TestLED3: now reaches U1.28 (P7.6)
- net TestLED3: now also R9.2
- net TestLED4: now reaches U1.29 (P7.7)
- net TestLED4: now also R10.2
- net SDA0: now reaches U1.35 (P3.3)
- net SDA0: now also P3.19 (P19), P4.19 (P19), P5.19 (P19), R13.2
- net SCL0: now reaches U1.36 (P3.4)
- net SCL0: now also P3.21 (P21), P4.21 (P21), P5.21 (P21), R14.2
- net HFXOUT: now reaches U1.85 (PJ.2)
- net HFXOUT: now also C10.1, Y2.2
- net HFXIN: now reaches U1.86 (PJ.3)
- net HFXIN: now also C9.1, Y2.1
- net TDI: now reaches U1.92 (PJ.4)
- net TDI: now also P2.10 (P10)
- net TDO_SWO: now reaches U1.93 (PJ.5)
- net TDO_SWO: now also P2.9 (P9)
- net at P3.35 (P35): now also D3.2 (A); no longer D3.1 (K)
- net at P3.36 (P36): now also R4.2; no longer R4.1
- net at P4.35 (P35): now also D4.2 (A); no longer D4.1 (K)
- net at P5.35 (P35): now also D5.2 (A); no longer D5.1 (K)
- net at R6.2: now also D5.1 (K); no longer D5.2 (A)
- net at R5.2: now also D4.1 (K); no longer D4.2 (A)
- removed net RX2: P3.31 (P31), P4.31 (P31), P5.31 (P31)
- removed net TX2: P3.33 (P33), P4.33 (P33), P5.33 (P33)
- new net: D3.1 (K), R4.1
- new net: D6.1 (K), R7.1
- new net: D7.1 (K), R8.1
- new net: D8.1 (K), R9.1
- new net: D9.1 (K), R10.1
- no-connect marks 30 -> 116
Other:
- note added: "380C (740F) <3sec"
- note added: "Monitoring"
- moved on the sheet: C1, C2, C3, C4, C5, C6, C7, C8, D1, D2, D3, D4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

Commit message: Start layout of motherboard
Parts:
- Y1: footprint (none) -> Crystals:Crystal_Round_Horizontal_3mm
- Y2: footprint (none) -> Crystals:Crystal_HC49-SD_SMD
Changed lines of the file:
@@
 F 0 "Y1" H 7200 5350 50  0000 C CNN
 F 1 "32.768khz" H 7200 5050 50  0000 C CNN
-F 2 "" H 7200 5200 50  0001 C CNN
+F 2 "Crystals:Crystal_Round_Horizontal_3mm" H 7200 5200 50  0001 C CNN
 F 3 "" H 7200 5200 50  0000 C CNN
 F 4 "http://www.digikey.com/product-detail/en/abracon-llc/AB38T-32.768KHZ/535-9034-ND/675229" H 7200 5200 60  0001 C CNN "Digikey"
@@
 F 0 "Y2" H 8850 5350 50  0000 C CNN
 F 1 "48MHz" H 8850 5050 50  0000 C CNN
-F 2 "" H 8850 5200 50  0001 C CNN
+F 2 "Crystals:Crystal_HC49-SD_SMD" H 8850 5200 50  0001 C CNN
 F 3 "" H 8850 5200 50  0000 C CNN
 F 4 "http://www.digikey.com/product-detail/en/ecs-inc/ECS-480-20-5P-TR/XC941CT-ND/465130" H 8850 5200 60  0001 C CNN "Digikey"

Commit message: Finish Mobo v1.0
Add XT60 power conector, add mounting holes, finish layout of
Motherboard v1.0
Parts:
- added P6: 12v POWER, XT60:XT60, symbol CONN_01X02
Connections:
- net +12V: now also P6.1 (P1)
- net GND: now also P6.2 (P2)
Changed lines of the file:
@@
 Connection ~ 6500 4200
 Wire Wire Line
-	900  6850 900  6750
+	900  6750 900  6850
 Wire Wire Line
 	850  6800 900  6800
@@
 	3700 1550 3700 1450
 Connection ~ 3700 1450
+$Comp
+L CONN_01X02 P6
+U 1 1 58742B22
+P 6300 1150
+F 0 "P6" H 6300 1300 50  0000 C CNN
+F 1 "12v POWER" V 6400 1150 50  0000 C CNN
+F 2 "XT60:XT60" H 6300 1150 50  0001 C CNN
+F 3 "" H 6300 1150 50  0000 C CNN
+	1    6300 1150
+	1    0    0    -1
+$EndComp
+$Comp
+L +12V #PWR052
+U 1 1 5874302E
+P 5900 1050
+F 0 "#PWR052" H 5900 900 50  0001 C CNN
+F 1 "+12V" H 5900 1190 50  0000 C CNN
+F 2 "" H 5900 1050 50  0000 C CNN
+F 3 "" H 5900 1050 50  0000 C CNN
+	1    5900 1050
+	1    0    0    -1
+$EndComp
+Wire Wire Line
+	5900 1050 5900 1100
+Wire Wire Line
+	5900 1100 6100 1100
+$Comp
+L GND #PWR053
+U 1 1 587431A1
+P 5900 1250
+F 0 "#PWR053" H 5900 1000 50  0001 C CNN
+F 1 "GND" H 5900 1100 50  0000 C CNN
+F 2 "" H 5900 1250 50  0000 C CNN
+F 3 "" H 5900 1250 50  0000 C CNN
+	1    5900 1250
+	1    0    0    -1
+$EndComp
+Wire Wire Line
+	5900 1200 6100 1200
+Wire Wire Line
+	5900 1200 5900 1250
 $EndSCHEMATC
